File: hw/sch_pcb/ADCoctoSPI01B.kicad_pcb (KiCad board)
At the start: 2 copper layers, 70.6 x 70.6 mm, 80 parts, among them J1 SATA7-67491-1030, J10 SAS_mini_1888174, J11 +5V, J2 SATA7-67491-1030, J3 SATA7-67491-1030, J4 SATA7-67491-1030, J5 HEADER_1x02, J6 HEADER_1x02, J7 SATA7-67491-1030, J8 HEADER_2x04, J9 HEADER_1x02, M1 HOLE, M2 HOLE, M3 HOLE, M4 HOLE, U1 AFE5801, U2 LM1117MP-1,8/NO, U3 LM1117MP-3,3/NO

Commit message: Edit PCB
Other:
- rule pad_to_mask_clearance: 0.15 -> 0.2
Changed lines of the file:
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@@
       (dielectric_constraints no)
     )
-    (pad_to_mask_clearance 0.15)
+    (pad_to_mask_clearance 0.2)
     (pcbplotparams
       (layerselection 0x0000030_80000001)
@@
     (pts (xy 130.556 136.906) (xy 130.556 66.294))
     (height 18.542)
-    (gr_text "2.7800 palec" (at 147.298 101.6 90) (layer "Dwgs.User")
+    (gr_text "2.7800 in" (at 147.298 101.6 90) (layer "Dwgs.User")
       (effects (font (size 1.5 1.5) (thickness 0.3)))
     )
@@
     (pts (xy 130.556 66.294) (xy 59.944 66.294))
     (height 17.272)
-    (gr_text "2.7800 palec" (at 95.25 47.222) (layer "Dwgs.User")
+    (gr_text "2.7800 in" (at 95.25 47.222) (layer "Dwgs.User")
       (effects (font (size 1.5 1.5) (thickness 0.3)))
     )
@@
     (pts (xy 125.73 71.12) (xy 64.77 71.12))
     (height 13.462)
-    (gr_text "2.4000 palec" (at 95.25 55.858) (layer "Dwgs.User")
+    (gr_text "2.4000 in" (at 95.25 55.858) (layer "Dwgs.User")
       (effects (font (size 1.5 1.5) (thickness 0.3)))
     )
@@
     (pts (xy 125.73 132.08) (xy 125.73 71.12))
     (height 15.24)
-    (gr_text "2.4000 palec" (at 139.17 101.6 90) (layer "Dwgs.User")
+    (gr_text "2.4000 in" (at 139.17 101.6 90) (layer "Dwgs.User")
       (effects (font (size 1.5 1.5) (thickness 0.3)))
     )
