File: hw/sch_pcb/ADCoctoSPI01B.kicad_sch (KiCad schematic)
At the start: 80 parts, among them J1 SATA7-67491-1030, J10 SAS_mini_1888174, J11 +5V, J2 SATA7-67491-1030, J3 SATA7-67491-1030, J4 SATA7-67491-1030, J5 HEADER_1x02, J6 HEADER_1x02, J7 SATA7-67491-1030, J8 HEADER_2x04, J9 HEADER_1x02, M1 HOLE, M2 HOLE, M3 HOLE, M4 HOLE, U1 AFE5801, U2 LM1117MP-1,8/NO, U3 LM1117MP-3,3/NO

Commit message: Příprava podkladů pro osazení
Parts:
- C1, C10, C11, C12, C13, C14, C15, C16, C2, C3, C4, C5, C6, C7, C8, C9: value 10nF -> (none); footprint Capacitor_SMD:C_0603_1608Metric -> (none)
- C17, C18, C19, C20, C21, C22, C23, C24, C25, C26, C27, C28, C29, C30, C32, C33, C34, C35, C36: value 100nF -> (none); footprint Capacitor_SMD:C_0603_1608Metric -> (none)
- C31: value 100uF/6V3 -> (none); footprint Capacitor_SMD:C_1210_3225Metric_Pad1.33x2.70mm_HandSolder -> (none)
- C37, C38: value 10uF -> (none); footprint Capacitor_SMD:C_0805_2012Metric -> (none)
- D1: value M4 -> (none); footprint Diode_SMD:D_SMA -> (none)
- J1, J2, J3, J4, J7: value SATA7-67491-1030 -> (none); footprint Mlab_CON:SATA-7_THT_VERT_2 -> (none)
- J10: value SAS_mini_1888174 -> (none); footprint Connector_SATA_SAS:SAS-mini_TEConnectivity_1888174_Vertical -> (none)
- J11: value +5V -> (none); footprint Mlab_Pin_Headers:Straight_2x03 -> (none)
- J5, J6, J9: value HEADER_1x02 -> (none); footprint Mlab_Pin_Headers:Straight_1x02 -> (none)
- J8: value HEADER_2x04 -> (none); footprint Mlab_Pin_Headers:Straight_2x04 -> (none)
- JP1: value SolderJumper_2_Bridged -> (none); footprint NetTie:NetTie-2_SMD_Pad0.5mm -> (none)
- L1, L2, L3: value BLM21PG300SN1D -> (none); footprint Inductor_SMD:L_0805_2012Metric_Pad1.15x1.40mm_HandSolder -> (none)
- M1, M2, M3, M4: value HOLE -> (none); footprint Mlab_Mechanical:MountingHole_3mm -> (none)
- R1, R19, R2, R3, R4, R5, R6, R7, R8: value 100 -> (none); footprint Resistor_SMD:R_0603_1608Metric -> (none)
- R10, R9: value 130 -> (none); footprint Resistor_SMD:R_0603_1608Metric -> (none)
- R11, R12, R13, R16, R17, R18: value 10k -> (none); footprint Resistor_SMD:R_0603_1608Metric -> (none)
- R14, R15: value 82 -> (none); footprint Resistor_SMD:R_0603_1608Metric -> (none)
- U1: value AFE5801 -> (none); footprint Mlab_IO:VQFN-64_9.15x9.15mm_EP_7.5x7.5mm -> (none)
- U2: value LM1117MP-1,8/NO -> (none); footprint Package_TO_SOT_SMD:SOT-223-3_TabPin2 -> (none)
- U3: value LM1117MP-3,3/NO -> (none); footprint Package_TO_SOT_SMD:SOT-223-3_TabPin2 -> (none)

Commit message: cleanup traces in schematics.
Parts:
- C1, C10, C11, C12, C13, C14, C15, C16, C2, C3, C4, C5, C6, C7, C8, C9: value (none) -> 10nF; footprint (none) -> Capacitor_SMD:C_0603_1608Metric
- C17, C18, C19, C20, C21, C22, C23, C24, C25, C26, C27, C28, C29, C30, C32, C33, C34, C35, C36: value (none) -> 100nF; footprint (none) -> Capacitor_SMD:C_0603_1608Metric
- C31: value (none) -> 100uF/6V3; footprint (none) -> Capacitor_SMD:C_1210_3225Metric_Pad1.33x2.70mm_HandSolder
- C37, C38: value (none) -> 10uF; footprint (none) -> Capacitor_SMD:C_0805_2012Metric
- D1: value (none) -> M4; footprint (none) -> Diode_SMD:D_SMA
- J1, J2, J3, J4, J7: value (none) -> SATA7-67491-1030; footprint (none) -> Mlab_CON:SATA-7_THT_VERT_2
- J10: value (none) -> SAS_mini_1888174; footprint (none) -> Connector_SATA_SAS:SAS-mini_TEConnectivity_1888174_Vertical
- J11: value (none) -> +5V; footprint (none) -> Mlab_Pin_Headers:Straight_2x03
- J5, J6, J9: value (none) -> HEADER_1x02; footprint (none) -> Mlab_Pin_Headers:Straight_1x02
- J8: value (none) -> HEADER_2x04; footprint (none) -> Mlab_Pin_Headers:Straight_2x04
- JP1: value (none) -> SolderJumper_2_Bridged; footprint (none) -> NetTie:NetTie-2_SMD_Pad0.5mm
- L1, L2, L3: value (none) -> BLM21PG300SN1D; footprint (none) -> Inductor_SMD:L_0805_2012Metric_Pad1.15x1.40mm_HandSolder
- M1, M2, M3, M4: value (none) -> HOLE; footprint (none) -> Mlab_Mechanical:MountingHole_3mm
- R1, R19, R2, R3, R4, R5, R6, R7, R8: value (none) -> 100; footprint (none) -> Resistor_SMD:R_0603_1608Metric
- R10, R9: value (none) -> 130; footprint (none) -> Resistor_SMD:R_0603_1608Metric
- R11, R12, R13, R16, R17, R18: value (none) -> 10k; footprint (none) -> Resistor_SMD:R_0603_1608Metric
- R14, R15: value (none) -> 82; footprint (none) -> Resistor_SMD:R_0603_1608Metric
- U1: value (none) -> AFE5801; footprint (none) -> Mlab_IO:VQFN-64_9.15x9.15mm_EP_7.5x7.5mm
- U2: value (none) -> LM1117MP-1,8/NO; footprint (none) -> Package_TO_SOT_SMD:SOT-223-3_TabPin2
- U3: value (none) -> LM1117MP-3,3/NO; footprint (none) -> Package_TO_SOT_SMD:SOT-223-3_TabPin2

Commit message: Cleanup schematics.
Changed lines of the file:
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@@
   (junction (at 222.25 90.805) (diameter 0.9144) (color 0 0 0 0)
   )
-  (junction (at 99.695 63.5) (diameter 0) (color 0 0 0 0)
-  )
   (junction (at 247.015 69.85) (diameter 0.9144) (color 0 0 0 0)
   )
@@
   (junction (at 91.44 176.53) (diameter 0.9144) (color 0 0 0 0)
   )
-  (junction (at 84.455 63.5) (diameter 0) (color 0 0 0 0)
-  )
   (junction (at 50.165 130.81) (diameter 0.9144) (color 0 0 0 0)
   )
@@
   (junction (at 50.165 110.49) (diameter 0.9144) (color 0 0 0 0)
   )
-  (junction (at 92.075 63.5) (diameter 0) (color 0 0 0 0)
-  )
   (junction (at 109.855 36.83) (diameter 0.9144) (color 0 0 0 0)
   )
@@
     (stroke (width 0) (type solid) (color 0 0 0 0))
   )
-  (wire (pts (xy 99.06 63.5) (xy 99.695 63.5))
-    (stroke (width 0) (type default) (color 0 0 0 0))
-  )
   (wire (pts (xy 198.755 90.17) (xy 200.025 90.17))
     (stroke (width 0) (type solid) (color 0 0 0 0))
@@
     (stroke (width 0) (type solid) (color 0 0 0 0))
   )
-  (wire (pts (xy 84.455 63.5) (xy 85.09 63.5))
-    (stroke (width 0) (type default) (color 0 0 0 0))
-  )
   (wire (pts (xy 127.635 16.51) (xy 122.555 16.51))
     (stroke (width 0) (type solid) (color 0 0 0 0))
@@
     (stroke (width 0) (type solid) (color 0 0 0 0))
   )
-  (wire (pts (xy 83.82 63.5) (xy 84.455 63.5))
-    (stroke (width 0) (type default) (color 0 0 0 0))
-  )
   (wire (pts (xy 120.015 29.845) (xy 126.365 29.845))
     (stroke (width 0) (type solid) (color 0 0 0 0))
@@
     (stroke (width 0) (type solid) (color 0 0 0 0))
   )
-  (wire (pts (xy 99.695 63.5) (xy 100.33 63.5))
-    (stroke (width 0) (type default) (color 0 0 0 0))
-  )
   (wire (pts (xy 160.655 118.11) (xy 177.165 118.11))
     (stroke (width 0) (type solid) (color 0 0 0 0))
@@
     (stroke (width 0) (type solid) (color 0 0 0 0))
   )
-  (wire (pts (xy 91.44 63.5) (xy 92.075 63.5))
-    (stroke (width 0) (type default) (color 0 0 0 0))
-  )
   (wire (pts (xy 200.025 140.97) (xy 200.025 148.59))
     (stroke (width 0) (type solid) (color 0 0 0 0))
@@
     (stroke (width 0) (type solid) (color 0 0 0 0))
   )
-  (wire (pts (xy 92.075 63.5) (xy 92.71 63.5))
-    (stroke (width 0) (type default) (color 0 0 0 0))
-  )
   (wire (pts (xy 200.025 74.93) (xy 200.025 82.55))
     (stroke (width 0) (type solid) (color 0 0 0 0))
@@
     (stroke (width 0) (type solid) (color 0 0 0 0))
   )
-  (text "Bias1" (at 59.69 162.56 0)
+  (text "Bias1" (at 62.23 162.56 0)
     (effects (font (size 1.524 1.524)) (justify left bottom))
   )
@@
   (symbol (lib_id "ADCoctoSPI01A-rescue:SATA7-67491-1030-MLAB_CONNECTORS") (at 36.195 81.28 180) (unit 1)
     (in_bom yes) (on_board yes)
-    (property "Reference" "J1" (id 0) (at 38.735 91.44 0)
+    (property "Reference" "J1" (id 0) (at 29.21 80.645 0)
       (effects (font (size 1.27 1.27)) (justify left bottom))
     )
@@
   (symbol (lib_id "ADCoctoSPI01A-rescue:SATA7-67491-1030-MLAB_CONNECTORS") (at 36.195 101.6 180) (unit 1)
     (in_bom yes) (on_board yes)
-    (property "Reference" "J2" (id 0) (at 38.735 111.76 0)
+    (property "Reference" "J2" (id 0) (at 29.21 100.965 0)
       (effects (font (size 1.27 1.27)) (justify left bottom))
     )
@@
   (symbol (lib_id "ADCoctoSPI01A-rescue:SATA7-67491-1030-MLAB_CONNECTORS") (at 36.195 121.92 180) (unit 1)
     (in_bom yes) (on_board yes)
-    (property "Reference" "J3" (id 0) (at 38.735 132.08 0)
+    (property "Reference" "J3" (id 0) (at 29.21 121.285 0)
       (effects (font (size 1.27 1.27)) (justify left bottom))
     )
@@
   (symbol (lib_id "ADCoctoSPI01A-rescue:SATA7-67491-1030-MLAB_CONNECTORS") (at 36.195 142.24 180) (unit 1)
     (in_bom yes) (on_board yes)
-    (property "Reference" "J4" (id 0) (at 38.735 152.4 0)
+    (property "Reference" "J4" (id 0) (at 29.21 144.145 0)
       (effects (font (size 1.27 1.27)) (justify left bottom))
     )
@@
   (symbol (lib_id "ADCoctoSPI01A-rescue:C_Small-device") (at 81.28 163.83 180) (unit 1)
     (in_bom yes) (on_board yes)
-    (property "Reference" "C17" (id 0) (at 78.74 163.83 90)
+    (property "Reference" "C17" (id 0) (at 78.74 161.29 90)
       (effects (font (size 1.27 1.27)) (justify left))
     )
@@
   (symbol (lib_id "ADCoctoSPI01A-rescue:HEADER_1x02-MLAB_HEADER") (at 71.12 161.29 0) (mirror y) (unit 1)
     (in_bom yes) (on_board yes)
-    (property "Reference" "J5" (id 0) (at 69.1388 161.163 0)
+    (property "Reference" "J5" (id 0) (at 72.39 157.48 0)
       (effects (font (size 1.524 1.524)) (justify left))
     )
@@
     (pin "1")
   )
-  (symbol (lib_id "power:GNDA") (at 100.33 63.5 180) (unit 1)
+  (symbol (lib_id "power:GNDA") (at 99.695 63.5 180) (unit 1)
     (in_bom yes) (on_board yes)
-    (property "Reference" "#PWR025" (id 0) (at 100.33 57.15 0)
+    (property "Reference" "#PWR025" (id 0) (at 99.695 57.15 0)
       (effects (font (size 1.27 1.27)) hide)
     )
-    (property "Value" "GNDA" (id 1) (at 100.33 59.69 0))
-    (property "Footprint" "" (id 2) (at 100.33 63.5 0)
+    (property "Value" "GNDA" (id 1) (at 99.695 59.69 0))
+    (property "Footprint" "" (id 2) (at 99.695 63.5 0)
       (effects (font (size 1.27 1.27)) hide)
     )
-    (property "Datasheet" "" (id 3) (at 100.33 63.5 0)
+    (property "Datasheet" "" (id 3) (at 99.695 63.5 0)
       (effects (font (size 1.27 1.27)) hide)
     )
     (pin "1")
   )
-  (symbol (lib_id "power:GNDA") (at 92.71 63.5 180) (unit 1)
+  (symbol (lib_id "power:GNDA") (at 92.075 63.5 180) (unit 1)
     (in_bom yes) (on_board yes)
-    (property "Reference" "#PWR019" (id 0) (at 92.71 57.15 0)
+    (property "Reference" "#PWR019" (id 0) (at 92.075 57.15 0)
       (effects (font (size 1.27 1.27)) hide)
     )
-    (property "Value" "GNDA" (id 1) (at 92.71 59.69 0))
-    (property "Footprint" "" (id 2) (at 92.71 63.5 0)
+    (property "Value" "GNDA" (id 1) (at 92.075 59.69 0))
+    (property "Footprint" "" (id 2) (at 92.075 63.5 0)
       (effects (font (size 1.27 1.27)) hide)
     )
-    (property "Datasheet" "" (id 3) (at 92.71 63.5 0)
+    (property "Datasheet" "" (id 3) (at 92.075 63.5 0)
       (effects (font (size 1.27 1.27)) hide)
     )
@@
     (pin "1")
   )
-  (symbol (lib_id "power:GNDA") (at 85.09 63.5 180) (unit 1)
+  (symbol (lib_id "power:GNDA") (at 84.455 63.5 180) (unit 1)
     (in_bom yes) (on_board yes)
-    (property "Reference" "#PWR017" (id 0) (at 85.09 57.15 0)
+    (property "Reference" "#PWR017" (id 0) (at 84.455 57.15 0)
       (effects (font (size 1.27 1.27)) hide)
     )
-    (property "Value" "GNDA" (id 1) (at 85.09 59.69 0))
-    (property "Footprint" "" (id 2) (at 85.09 63.5 0)
+    (property "Value" "GNDA" (id 1) (at 84.455 59.69 0))
+    (property "Footprint" "" (id 2) (at 84.455 63.5 0)
       (effects (font (size 1.27 1.27)) hide)
     )
-    (property "Datasheet" "" (id 3) (at 85.09 63.5 0)
+    (property "Datasheet" "" (id 3) (at 84.455 63.5 0)
       (effects (font (size 1.27 1.27)) hide)
     )
